Commit message: corrected inertia in tag model

File: gazebo_rfid_node/urdf/tag_model.xacro (robot description, xacro)
@@ -25,5 +25,5 @@
     <mass value="1e-5" />
     <origin xyz="0 0 0" rpy="0 0 0"/>
-    <inertia ixx="1e-6" ixy="0" ixz="0" iyy="1e-6" iyz="0" izz="1e-6" />
+    <inertia ixx="1e-1" ixy="0" ixz="0" iyy="1e-1" iyz="0" izz="1e-1" />
   </inertial>
 </link>
