Commit message: Two antennas launch file and model

File: gazebo/gazebo_rfid_node/urdf/tag_model.xacro (robot description, xacro)
@@ -27,4 +27,10 @@
   </inertial>
 </link>
+<link name="world" />
+ <joint name="world_joint" type="fixed">
+    <parent link="world" />
+    <child link = "$(arg tf_prefix)/rfid_tag_$(arg ID)_link" />
+    <origin xyz="0.0 0.0 0.7" rpy="0.0 0.0 0.0" />
+ </joint>
 <gazebo reference="$(arg tf_prefix)/rfid_tag_$(arg ID)_link">
   <turnGravityOff>true</turnGravityOff>

Commit message: Remove static tag

File: gazebo/gazebo_rfid_node/urdf/tag_model.xacro (robot description, xacro)
@@ -27,10 +27,11 @@
   </inertial>
 </link>
-<link name="world" />
+<!-- enable the following to keep the model static -->
+<!-- <link name="world" />
  <joint name="world_joint" type="fixed">
     <parent link="world" />
     <child link = "$(arg tf_prefix)/rfid_tag_$(arg ID)_link" />
-    <origin xyz="0.0 0.0 0.7" rpy="0.0 0.0 0.0" />
- </joint>
+    <origin xyz="0.0 0.0 0.0" rpy="0.0 0.0 0.0" />
+ </joint> -->
 <gazebo reference="$(arg tf_prefix)/rfid_tag_$(arg ID)_link">
   <turnGravityOff>true</turnGravityOff>
