Commit message: Added standing_person model and fix mesh loading

File: gazebo/gazebo_rfid_node/urdf/person_tag_model.xacro (robot description, xacro)
@@ -26,5 +26,5 @@
     <origin xyz="0 0 0" rpy="0 0 0"/>
     <geometry>
-      <mesh filename="package://rasberry_gazebo/models/rfid_person/meshes/standing.dae"/>
+      <mesh filename="package://gazebo_rfid_node/models/person_standing/meshes/standing.dae"/>
     </geometry>
   </collision>
@@ -32,5 +32,5 @@
     <pose>0 0 0.02 0.04 0 0</pose>
     <geometry>
-      <mesh filename="package://rasberry_gazebo/models/rfid_person/meshes/standing.dae"/>
+      <mesh filename="package://gazebo_rfid_node/models/person_standing/meshes/standing.dae"/>
     </geometry>
   </visual>

Commit message: Fix collision in human model

File: gazebo/gazebo_rfid_node/urdf/person_tag_model.xacro (robot description, xacro)
@@ -9,11 +9,24 @@
 <!-- person -->
 <link name="$(arg tf_prefix)/person">
-  <!-- <static>1</static> -->
   <inertial>
-    <origin xyz="0 0 0" rpy="0 0 0"/>
+    <origin xyz="0 -0.1 0.95" rpy="0 0 0"/>
     <mass value="80" />
     <inertia ixx="24.88" ixy="0" ixz="0" iyy="25.73" iyz="0" izz="2.48" />
   </inertial>
-  <collision name="bottom">
+  <collision name="$(arg tf_prefix)/person_collision">
+    <origin xyz="0 0 0.02" rpy="0.04 0 0"/>
+    <geometry>
+      <mesh scale="1 1 1" filename="package://gazebo_rfid_node/models/person_standing/meshes/standing.dae"/>
+    </geometry>
+  </collision>
+  <visual name="visual">
+    <origin xyz="0 0 0.02" rpy="0.04 0 0"/>
+    <geometry>
+      <mesh filename="package://gazebo_rfid_node/models/person_standing/meshes/standing.dae"/>
+    </geometry>
+  </visual>
+</link>
+<link name="$(arg tf_prefix)/bottom">
+  <collision name="$(arg tf_prefix)/bottom_collision">
     <origin xyz="0 0 0" rpy="0 0 0"/>
     <geometry>
@@ -23,16 +36,17 @@
     </geometry>
   </collision>
-  <collision name="person">
+  <inertial>
     <origin xyz="0 0 0" rpy="0 0 0"/>
+    <mass value="80" />
+    <inertia ixx="24.88" ixy="0" ixz="0" iyy="25.73" iyz="0" izz="2.48" />
+  </inertial>
+  <!-- <visual name="visual">
+    <origin xyz="0 0 0.02" rpy="0.04 0 0"/>
     <geometry>
-      <mesh filename="package://gazebo_rfid_node/models/person_standing/meshes/standing.dae"/>
+      <box>
+        <size>0.5 0.35 0.02</size>
+      </box>
     </geometry>
-  </collision>
-  <visual name="visual">
-    <pose>0 0 0.02 0.04 0 0</pose>
-    <geometry>
-      <mesh filename="package://gazebo_rfid_node/models/person_standing/meshes/standing.dae"/>
-    </geometry>
-  </visual>
+  </visual> -->
 </link>
 <!-- RFID reader -->
@@ -56,4 +70,9 @@
   </inertial>
 </link>
+<joint name="bottom_person" type="fixed">
+  <parent link="$(arg tf_prefix)/person"/>
+  <child link="$(arg tf_prefix)/bottom"/>
+  <origin xyz="0 -0.1 0.01" rpy="0.0 0.0 0" />
+</joint>
 <joint name="link_rfid" type="fixed">
   <parent link="$(arg tf_prefix)/person"/>
@@ -61,11 +80,4 @@
   <origin xyz="-0.27 -0.05 1.4" rpy="0.0 0.0 0" />  <!-- tag on the arm below the shoulder-->
 </joint>
-<!-- enable the following to keep the model static -->
-<!-- <link name="world" />
- <joint name="world_joint" type="fixed">
-    <parent link="world" />
-    <child link = "$(arg tf_prefix)/rfid_tag_$(arg ID)_link" />
-    <origin xyz="0.0 0.0 0.7" rpy="0.0 0.0 0.0" />
- </joint> -->
 <gazebo reference="$(arg tf_prefix)/rfid_tag_$(arg ID)_link">
   <turnGravityOff>true</turnGravityOff>

Commit message: Identify people by ID + fix reference frame

File: gazebo/gazebo_rfid_node/urdf/person_tag_model.xacro (robot description, xacro)
@@ -8,5 +8,5 @@
 <xacro:arg name="tf_prefix" default=""/>
 <!-- person -->
-<link name="$(arg tf_prefix)/person">
+<link name="$(arg tf_prefix)/person_$(arg ID)">
   <inertial>
     <origin xyz="0 -0.1 0.95" rpy="0 0 0"/>
@@ -27,5 +27,5 @@
   </visual>
 </link>
-<link name="$(arg tf_prefix)/bottom">
+<link name="$(arg tf_prefix)/bottom_$(arg ID)">
   <collision name="$(arg tf_prefix)/bottom_collision">
     <origin xyz="0 0 0" rpy="0 0 0"/>
@@ -71,10 +71,10 @@
 </link>
 <joint name="bottom_person" type="fixed">
-  <parent link="$(arg tf_prefix)/person"/>
-  <child link="$(arg tf_prefix)/bottom"/>
+  <parent link="$(arg tf_prefix)/person_$(arg ID)"/>
+  <child link="$(arg tf_prefix)/bottom_$(arg ID)"/>
   <origin xyz="0 -0.1 0.01" rpy="0.0 0.0 0" />
 </joint>
 <joint name="link_rfid" type="fixed">
-  <parent link="$(arg tf_prefix)/person"/>
+  <parent link="$(arg tf_prefix)/person_$(arg ID)"/>
   <child link="$(arg tf_prefix)/rfid_tag_$(arg ID)_link"/>
   <origin xyz="-0.27 -0.05 1.4" rpy="0.0 0.0 0" />  <!-- tag on the arm below the shoulder-->
@@ -98,5 +98,5 @@
   <plugin name="ground_truth" filename="libgazebo_ros_p3d.so">
     <frameName>map</frameName>
-    <bodyName>$(arg tf_prefix)/rfid_tag_$(arg ID)_link</bodyName>
+    <bodyName>$(arg tf_prefix)/person_$(arg ID)</bodyName>
     <topicName>poses/$(arg ID)</topicName>
     <updateRate>5.0</updateRate>
